Commit message: Roarm M2 adds a gripper.

File: public/URDF/roarm_m2.urdf (robot description, URDF)
Before this commit: robot roarm_m2, 7 links, 6 joints
Links:
- added link gripper_base, mass 0.0144765; collision mesh filename=meshes/gripper/gripper_base.stl; visual mesh filename=meshes/gripper/gripper_base.stl
- link gripper_link: geometry collision mesh filename=meshes/gripper/gripper_link.stl; visual mesh filename=meshes/gripper/gripper_link.stl
- link link3: mass 0.0269773 -> 0.0181535
Joints:
- removed joint link3_to_gripper_link
- added joint gripper_joint: type revolute, parent gripper_base, child gripper_link, origin xyz=0 0 0 rpy=0 0 0, axis 0 0 -1, limit lower=0 upper=1.57 effort=1000.0 velocity=0.5
- added joint link3_to_gripper_base: type fixed, parent link3, child gripper_base, origin xyz=0.002906 -0.21599 -0.00066683 rpy=1.5708 0 -1.5708, axis 0 0 1
- joint link2_to_link3: origin xyz=0.236815132922094 0.0300023995170449 0 rpy=0 0 1.5708 -> xyz=0.236774 0.0300023995170449 0 rpy=0 0 1.5708
